Commit message: Foot STL text -> binary

File: URDF/roid1_12dof.urdf (robot description, URDF)
Before this commit: robot Roid1, 25 links, 24 joints
Joints:
- joint c_chest_yaw: type revolute -> fixed
- joint c_head_yaw: type revolute -> fixed
- joint l_elbow_pitch: type revolute -> fixed
- joint l_elbow_yaw: type revolute -> fixed
- joint l_shoulder_pitch: type revolute -> fixed
- joint l_shoulder_roll: type revolute -> fixed
- joint r_elbow_pitch: type revolute -> fixed
- joint r_elbow_yaw: type revolute -> fixed
- joint r_shoulder_pitch: type revolute -> fixed
- joint r_shoulder_roll: type revolute -> fixed

File: URDF/roid1_urdf_12dof.urdf (robot description, URDF)
Before this commit: robot Roid1, 25 links, 24 joints
Links:
- link base_link: geometry collision mesh filename=package://roid1/URDF/roid1_description/meshes/c_waist.stl; visual mesh filename=package://roid1/URDF/roid1_description/meshes/c_waist.stl
- link c_chest: geometry visual mesh filename=package://roid1/URDF/roid1_description/meshes/c_chest.stl
- link c_chest_c: geometry collision mesh filename=package://roid1/URDF/roid1_description/meshes/c_chest_b.stl; visual mesh filename=package://roid1/URDF/roid1_description/meshes/c_chest_b.stl
- link c_head: geometry collision mesh filename=package://roid1/URDF/roid1_description/meshes/c_head_a.stl; visual mesh filename=package://roid1/URDF/roid1_description/meshes/c_head_a.stl
- link l_ankle: geometry collision mesh filename=package://roid1/URDF/roid1_description/meshes/l_ankle.stl; visual mesh filename=package://roid1/URDF/roid1_description/meshes/l_ankle.stl
- link l_elbow: geometry collision mesh filename=package://roid1/URDF/roid1_description/meshes/l_elbow.stl; visual mesh filename=package://roid1/URDF/roid1_description/meshes/l_elbow.stl
- link l_foot: geometry collision mesh filename=package://roid1/URDF/roid1_description/meshes/l_foot_middle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; visual mesh filename=package://roid1/URDF/roid1_description/meshes/l_foot_middle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
- link l_hipjoint_lower: geometry collision mesh filename=package://roid1/URDF/roid1_description/meshes/l_hipjoint_lo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; visual mesh filename=package://roid1/URDF/roid1_description/meshes/l_hipjoint_lo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
- link l_hipjoint_upper: geometry collision mesh filename=package://roid1/URDF/roid1_description/meshes/l_hipjoint_up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; visual mesh filename=package://roid1/URDF/roid1_description/meshes/dec_l_hipjoin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
- link l_leg_lower: geometry collision mesh filename=package://roid1/URDF/roid1_description/meshes/l_leg_lower_a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; collision mesh filename=package://roid1/URDF/roid1_description/meshes/l_leg_lower_b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
- link l_leg_upper: geometry collision mesh filename=package://roid1/URDF/roid1_description/meshes/l_leg_upper_a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; visual mesh filename=package://roid1/URDF/roid1_description/meshes/l_leg_upper_a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
- link l_lowerarm: geometry collision mesh filename=package://roid1/URDF/roid1_description/meshes/l_arm_lower.s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; visual mesh filename=package://roid1/URDF/roid1_description/meshes/l_arm_lower.s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
- link l_shoulder: geometry collision mesh filename=package://roid1/URDF/roid1_description/meshes/l_shoulder.stl; visual mesh filename=package://roid1/URDF/roid1_description/meshes/dec_shoulderp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
- link l_upperarm: geometry collision mesh filename=package://roid1/URDF/roid1_description/meshes/l_arm_upper.s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; visual mesh filename=package://roid1/URDF/roid1_description/meshes/l_arm_upper.s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
- link r_ankle: geometry collision mesh filename=package://roid1/URDF/roid1_description/meshes/r_ankle.stl; visual mesh filename=package://roid1/URDF/roid1_description/meshes/r_ankle.stl
- link r_elbow: geometry collision mesh filename=package://roid1/URDF/roid1_description/meshes/r_elbow.stl; visual mesh filename=package://roid1/URDF/roid1_description/meshes/r_elbow.stl
- link r_foot: geometry collision mesh filename=package://roid1/URDF/roid1_description/meshes/r_foot_middle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; visual mesh filename=package://roid1/URDF/roid1_description/meshes/r_foot_middle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
- link r_hipjoint_lower: geometry collision mesh filename=package://roid1/URDF/roid1_description/meshes/r_hipjoint_lo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; visual mesh filename=package://roid1/URDF/roid1_description/meshes/r_hipjoint_lo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
- link r_hipjoint_upper: geometry collision mesh filename=package://roid1/URDF/roid1_description/meshes/r_hipjoint_up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; visual mesh filename=package://roid1/URDF/roid1_description/meshes/dec_r_hipjoin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
- link r_leg_lower: geometry collision mesh filename=package://roid1/URDF/roid1_description/meshes/r_leg_lower_a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; collision mesh filename=package://roid1/URDF/roid1_description/meshes/r_leg_lower_b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
- link r_leg_upper: geometry collision mesh filename=package://roid1/URDF/roid1_description/meshes/r_leg_upper_a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; visual mesh filename=package://roid1/URDF/roid1_description/meshes/r_leg_upper_a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
- link r_lowerarm: geometry collision mesh filename=package://roid1/URDF/roid1_description/meshes/r_arm_lower.s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; visual mesh filename=package://roid1/URDF/roid1_description/meshes/r_arm_lower.s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
- link r_shoulder: geometry collision mesh filename=package://roid1/URDF/roid1_description/meshes/r_shoulder.stl; visual mesh filename=package://roid1/URDF/roid1_description/meshes/dec_shoulderp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
- link r_upperarm: geometry collision mesh filename=package://roid1/URDF/roid1_description/meshes/r_arm_upper.s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; visual mesh filename=package://roid1/URDF/roid1_description/meshes/r_arm_upper.s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
Joints:
- joint c_chest_yaw: type revolute -> fixed
- joint c_head_yaw: type revolute -> fixed
- joint l_elbow_pitch: type revolute -> fixed
- joint l_elbow_yaw: type revolute -> fixed
- joint l_shoulder_pitch: type revolute -> fixed
- joint l_shoulder_roll: type revolute -> fixed
- joint r_elbow_pitch: type revolute -> fixed
- joint r_elbow_yaw: type revolute -> fixed
- joint r_shoulder_pitch: type revolute -> fixed
- joint r_shoulder_roll: type revolute -> fixed
